Commit message: Setting proper joint limits and updating collision meshes

File: urdf/Dorna2.urdf (robot description, URDF)
Before this commit: robot Dorna_2_URDF, 6 links, 5 joints
Joints:
- joint Joint_0: limit lower=-2.7925 upper=3.1416 effort=10 velocity=10.472 -> lower=-3.0543 upper=3.1415 effort=10 velocity=10.472
- joint Joint_1: axis 0 1 0 -> 0 -1 0; limit lower=0 upper=4.7123 effort=10 velocity=7.854 -> lower=-1.5707 upper=3.1415 effort=10 velocity=7.854; origin xyz=0.095476 0.0508 0.20647 rpy=0 0 0 -> xyz=0.095476 0.0508 0.20647 rpy=0 -3.1415 0
- joint Joint_2: axis 0 1 0 -> 0 -1 0; limit lower=-4.9567 upper=0 effort=10 velocity=7.854 -> lower=-2.4783 upper=2.4783 effort=10 velocity=7.854; origin xyz=-0.20319 -0.00635 0.0022018 rpy=0 0 0 -> xyz=-0.20319 -0.00635 0.0022018 rpy=0 3.8048 0
- joint Joint_3: limit lower=-4.71239 upper=0 effort=10 velocity=34.907 -> lower=-2.3561 upper=2.3561 effort=10 velocity=34.907; origin xyz=0.1211 -0.007112 0.092521 rpy=0 0 0 -> xyz=0.1211 -0.007112 0.092521 rpy=0 -3.9268 0

Commit message: Change STL extension to stl because Blender always saves in .stl

File: urdf/Dorna2.urdf (robot description, URDF)
Before this commit: robot Dorna_2_URDF, 6 links, 5 joints
Links:
- link Link_1: geometry collision mesh filename=package://r2d2_urdf/meshes/Link_1_Collision.stl; visual mesh filename=package://r2d2_urdf/meshes/Link_1.stl
- link Link_2: geometry collision mesh filename=package://r2d2_urdf/meshes/Link_2_Collision.stl; visual mesh filename=package://r2d2_urdf/meshes/Link_2.stl
- link Link_3: geometry collision mesh filename=package://r2d2_urdf/meshes/Link_3_Collision.stl; visual mesh filename=package://r2d2_urdf/meshes/Link_3.stl
- link Link_4: geometry collision mesh filename=package://r2d2_urdf/meshes/Link_4_Collision.stl; visual mesh filename=package://r2d2_urdf/meshes/Link_4.stl
- link Link_5: geometry collision mesh filename=package://r2d2_urdf/meshes/Link_5_Collision.stl; visual mesh filename=package://r2d2_urdf/meshes/Link_5.stl
- link base_link: geometry collision mesh filename=package://r2d2_urdf/meshes/base_link_Collision.stl; visual mesh filename=package://r2d2_urdf/meshes/base_link.stl

Commit message: Fix rotation of Joint_4 as it rotated in the opposite direction

File: urdf/Dorna2.urdf (robot description, URDF)
Before this commit: robot Dorna_2_URDF, 6 links, 5 joints
Joints:
- joint Joint_4: axis 0.99117 0 -0.13261 -> -0.99117 0 0.13261
